File: ConstantCurrentTester.brd (EAGLE design)
At the start: 160 x 100 mm, 57 parts, among them J1 CONN_62.54, Q1 35A/25V/8.5mΩ, U1 ATMEGA328P_TQFP, U2 MCP4726A0SOT-23, U3 MCP6041, U4 INA219D, U5 SN74LVC1G3157SC70, U6 TLV61220DBV, U7 MCP6041, Y1 8MHz

Commit message: Adapted Schematic, layout ready for review/cleanup
Main layout complete, details and minor cleanup remain
Parts:
- removed R9: 1.0, rcl:0617/22
- added JP1: JUMPER-SMT_2_NC_PASTE_SILK, SparkFun-Jumpers:SMT-JUMPER_2_NC_PASTE_SILK
- added R18, R19: 2, bschulz_passives:R2512
- R10: device bschulz_passives:0207/10 -> bschulz_passives:R0603
- moved S3 202.6 mm to (58.0, 65.9), turned to 90 degrees
- moved R17 173.0 mm to (16.5, 27.9), turned to 90 degrees
- moved R13 170.8 mm to (15.2, 31.8)
- moved R16 169.2 mm to (14.0, 27.9), turned to 90 degrees
- moved U5 168.0 mm to (33.8, 31.6)
- moved R12 166.7 mm to (19.1, 26.7), turned to 270 degrees
- moved U7 164.9 mm to (19.1, 30.5)
- moved C11 157.4 mm to (47.0, 16.5), turned to 90 degrees
- moved R11 154.2 mm to (52.7, 11.4)
- moved RT1 153.3 mm to (19.1, 12.8), turned to 180 degrees
- moved U4 152.7 mm to (50.8, 17.8), turned to 180 degrees
- moved J2 144.1 mm to (54.6, 5.08)
- moved C10 131.2 mm to (25.4, 24.1), turned to 180 degrees
- moved C9 130.6 mm to (25.4, 26.7), turned to 180 degrees
- moved U3 128.0 mm to (30.5, 30.5)
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Connections:
- removed net N$4: R5.1, U$1.CD1
- removed net THERM_SENSE: U1.26
- removed net VCC: R1.2
- new net N$13: R18.1, R19.2
- new net V_BACKUP: BT1.POWER0, BT1.POWER1, U$2.3
- net 3V3: now also R1.2
- net FB: now also R18.2; no longer R9.2
- net GND: now also JP1.1, R19.1; no longer R9.1
- net LOAD: now also JP1.2
- net PWR_OVERRIDE: now also U1.26
- net SD_CD: now also R5.1, U$1.CD1
- net VBAT: no longer BT1.POWER0, BT1.POWER1, U$2.3
Routing:
- net GND: track 17.1 -> 521.3 mm, vias 3 -> 11
- net 3V3: track 8.46 -> 281.7 mm, vias 0 -> 6
- net SDA: track 0.00 -> 89.8 mm, vias 0 -> 4
- net SCL: track 0.00 -> 87.9 mm, vias 0 -> 4
- net !RESET: track 0.00 -> 67.9 mm
- net FB: track 0.00 -> 51.4 mm, vias 0 -> 2
- net PWR_OVERRIDE: track 0.00 -> 41.6 mm, vias 0 -> 3
- net MISO: track 0.00 -> 36.4 mm
- net REC: track 0.00 -> 35.3 mm
- net MOSI: track 0.00 -> 35.2 mm
- net LOAD: track 0.00 -> 34.7 mm, vias 0 -> 17
- net V_BACKUP: track 0.00 -> 34.2 mm
- net TX: track 0.00 -> 33.9 mm, vias 0 -> 1
- net VBAT: track 0.00 -> 31.8 mm
- net SCK: track 0.00 -> 31.3 mm, vias 0 -> 1
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- added copper zone on layer 1, net LOAD
- added copper zone on layer 16, net LOAD
Other:
- board size 160 x 100 mm -> 63.5 x 91.1 mm
- board text added: "+"
- board text added: "-"
- board text added: "3v3"
- board text added: "DTR"
- board text added: "FB"
- board text added: "GND"
- board text added: "Project Bast Bobby Schulz 01/28/2020 v0.0"
- board text added: "REC"
- board text added: "RESET"
- board text added: "RX"
- board text added: "Solar"
- board text added: "TX"
